File: HDK/template_project.kicad_sch (KiCad schematic)
At the start: 1 part, among them U101 STM32F072C8Tx

Commit message: updated docs
Other:
- added sheet Power (Power.kicad_sch)
Changed lines of the file:
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@@
+		)
+	)
+	(sheet
+		(at 116.84 43.18)
+		(size 15.24 12.7)
+		(fields_autoplaced yes)
+		(stroke
+			(width 0.1524)
+			(type solid)
+		)
+		(fill
+			(color 0 0 0 0.0000)
+		)
+		(property "Sheetname" "Power"
+			(at 116.84 42.4684 0)
+			(effects
+				(font
+					(size 1.27 1.27)
+				)
+				(justify left bottom)
+			)
+		)
+		(property "Sheetfile" "Power.kicad_sch"
+			(at 116.84 56.4646 0)
+			(effects
+				(font
+					(size 1.27 1.27)
+				)
+				(justify left top)
+			)
+		)
+		(instances
+			(project "template_project"
+				(path "/26f9cb6a-983b-4cfb-90f4-253f3e225603"
+					(page "2")
+				)
+			)
 		)
 	)
