File: HDK/Power.kicad_sch (KiCad schematic)
At the start: 1 part, among them U201 AMS1117

Commit message: updated docs workflow
Other:
- removed sheet Power Sub
- added sheet PowerSub (PowerSub.kicad_sch)
Changed lines of the file:
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@@
 	)
 	(sheet
-		(at 123.19 67.31)
-		(size 12.7 7.62)
+		(at 130.81 72.39)
+		(size 12.7 10.16)
 		(fields_autoplaced yes)
 		(stroke
@@
 			(color 0 0 0 0.0000)
 		)
-		(property "Sheetname" "Power Sub"
-			(at 123.19 66.5984 0)
+		(property "Sheetname" "PowerSub"
+			(at 130.81 71.6784 0)
 			(effects
 				(font
@@
 		)
 		(property "Sheetfile" "PowerSub.kicad_sch"
-			(at 123.19 75.5146 0)
+			(at 130.81 83.1346 0)
 			(effects
 				(font
